Commit message: 补充正确的质量信息Updated RM75-B URDF file to correct mesh file paths, added inertial properties for links, and refined joint dynamics for improved performance. Introduced new links and joints for gripper pads.

File: RM75+gripper/RM75-B/urdf/RM75-B.urdf (robot description, URDF)
Before this commit: robot RM75B_with_Gripper, 16 links, 15 joints
Links:
- added link left_pad, mass 0.01
- added link right_pad, mass 0.01
- link base_link: geometry collision mesh filename=../meshes/base_link.STL; visual mesh filename=../meshes/base_link.STL
- link gripper_Left_1_Link: mass None -> 0.05; geometry collision mesh filename=../../crt_ctag2f90d_gripper_visualization/meshes/Left_1_Lin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; visual mesh filename=../../crt_ctag2f90d_gripper_visualization/meshes/Left_1_Lin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
- link gripper_Left_2_Link: mass None -> 0.05; geometry collision mesh filename=../../crt_ctag2f90d_gripper_visualization/meshes/Left_2_Lin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; visual mesh filename=../../crt_ctag2f90d_gripper_visualization/meshes/Left_2_Lin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
- link gripper_Left_Support_Link: mass None -> 0.03; geometry collision mesh filename=../../crt_ctag2f90d_gripper_visualization/meshes/Left_Suppo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; visual mesh filename=../../crt_ctag2f90d_gripper_visualization/meshes/Left_Suppo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
- link gripper_Right_1_Link: mass None -> 0.05; geometry collision mesh filename=../../crt_ctag2f90d_gripper_visualization/meshes/Right_1_Li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; visual mesh filename=../../crt_ctag2f90d_gripper_visualization/meshes/Right_1_Li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
- link gripper_Right_2_Link: mass None -> 0.05; geometry collision mesh filename=../../crt_ctag2f90d_gripper_visualization/meshes/Right_2_Li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; visual mesh filename=../../crt_ctag2f90d_gripper_visualization/meshes/Right_2_Li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
- link gripper_Right_Support_Link: mass None -> 0.03; geometry collision mesh filename=../../crt_ctag2f90d_gripper_visualization/meshes/Right_Supp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; visual mesh filename=../../crt_ctag2f90d_gripper_visualization/meshes/Right_Supp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
- link gripper_base_link: mass None -> 0.15; geometry collision mesh filename=../../crt_ctag2f90d_gripper_visualization/meshes/base_link.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; visual mesh filename=../../crt_ctag2f90d_gripper_visualization/meshes/base_link.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
- link link_1: mass None -> 1.5; geometry collision mesh filename=../meshes/link_1.STL; visual mesh filename=../meshes/link_1.STL
- link link_2: mass None -> 1.2; geometry collision mesh filename=../meshes/link_2.STL; visual mesh filename=../meshes/link_2.STL
- link link_3: mass None -> 1.0; geometry collision mesh filename=../meshes/link_3.STL; visual mesh filename=../meshes/link_3.STL
- link link_4: mass None -> 0.8; geometry collision mesh filename=../meshes/link_4.STL; visual mesh filename=../meshes/link_4.STL
- link link_5: mass None -> 0.6; geometry collision mesh filename=../meshes/link_5.STL; visual mesh filename=../meshes/link_5.STL
- link link_6: mass None -> 0.3; geometry collision mesh filename=../meshes/link_6.STL; visual mesh filename=../meshes/link_6.STL
- link link_7: geometry collision mesh filename=../meshes/link_7.STL; visual mesh filename=../meshes/link_7.STL
Joints:
- added joint left_pad_joint: type fixed, parent gripper_Left_Support_Link, child left_pad, origin xyz=-0.02 0.055 0 rpy=0 0 0
- added joint right_pad_joint: type fixed, parent gripper_Right_Support_Link, child right_pad, origin xyz=-0.02 0.055 0 rpy=0 0 0
- joint arm_gripper_joint: origin xyz=0 0 0 rpy=0 0 0 -> xyz=0 0 0 rpy=0 0 0.5236
- joint gripper_Left_1_Joint: axis 0 0 -1 -> 0 0 1; limit lower=-0.91 upper=0 effort=10 velocity=10 -> lower=0 upper=0.91 effort=10 velocity=10
- joint gripper_Left_2_Joint: axis 0 0 -1 -> 0 0 1; limit lower=-3.14 upper=3.14 effort=10 velocity=10 -> lower=0 upper=0.91 effort=10 velocity=10; mimic joint=gripper_Left_1_Joint multiplier=1 offset=0 -> (none)
- joint gripper_Left_Support_Joint: limit lower=-3.14 upper=3.14 effort=10 velocity=10 -> lower=0 upper=0.91 effort=10 velocity=10; mimic joint=gripper_Left_1_Joint multiplier=-1 offset=0 -> (none)
- joint gripper_Right_1_Joint: limit lower=-3.14 upper=3.14 effort=10 velocity=10 -> lower=0 upper=0.91 effort=10 velocity=10; mimic joint=gripper_Left_1_Joint multiplier=-1 offset=0 -> (none)
- joint gripper_Right_2_Joint: limit lower=-3.14 upper=3.14 effort=10 velocity=10 -> lower=0 upper=0.91 effort=10 velocity=10; mimic joint=gripper_Left_1_Joint multiplier=-1 offset=0 -> (none)
- joint gripper_Right_Support_Joint: limit lower=-3.14 upper=3.14 effort=10 velocity=10 -> lower=0 upper=0.91 effort=10 velocity=10; mimic joint=gripper_Left_1_Joint multiplier=-1 offset=0 -> (none)
